Commit message: new changes for sim

File: description/robot.urdf.xacro (robot description, xacro)
@@ -1,4 +1,4 @@
 <?xml version="1.0"?>
 <robot xmlns:xacro="http://www.ros.org/wiki/xacro"  name="robot">
-<xacro:include filename="robot_core.xacro" />
+<xacro:include filename="SolidworksDesign.xacro" />
 </robot>

File: description/robot_core.xacro (robot description, xacro)
@@ -1,7 +1,11 @@
 <?xml version="1.0"?>
 <robot xmlns:xacro="http://www.ros.org/wiki/xacro" >
+<xacro:include filename="inertial_macros.xacro"/>
     <material name="white">
         <color rgba="1 1 1 1" />
     </material>
+    <material name="pink">
+    <color rgba="1 0 1 1" /> <!-- Pink color with RGBA values -->
+</material>
     <material name="red">
         <color rgba="1 0 0 1" />
@@ -36,13 +40,25 @@
             <origin xyz="0.15 0.0 0.075" rpy="0.0 0.0 0.0"/>
             <geometry>
+              <mesh filename="package://firefighting_robot/meshes/base_link.STL" scale="1.0"/>
+            </geometry>
+            <material name="pink"/>
+        </visual>
+        <collision>
+            <origin xyz="0.15 0.0 0.075" rpy="0.0 0.0 0.0"/>
+            <geometry>
                 <box size="0.3 0.3 0.15"/>
             </geometry>
-            <material name="white"/>
-        </visual>
+        </collision>
+        <xacro:inertial_box mass="0.5" x="0.3" y="0.3" z="0.15">
+            <origin xyz="0.15 0.0 0.075" rpy="0.0 0.0 0.0"/>
+        </xacro:inertial_box>
     </link>
+    <gazebo reference="chassis">
+        <material>Gazebo/Red</material>
+    </gazebo>
     <joint name="left_wheel_joint" type="continuous">
-        <parent link="base_link"/>
+        <parent link="chassis"/>
         <child link="left_wheel"/>
-        <origin xyz="0.0 0.175 0.0" rpy="-${pi/2} 0.0 0.0"/>
+        <origin xyz="0.03 0.175 0.0" rpy="-${pi/2} 0.0 0.0"/>
         <axis xyz="0.0 0.0 1"/>
     </joint>
@@ -54,9 +70,20 @@
             <material name="blue" />
         </visual>
+        <collision>
+            <geometry>
+                <cylinder radius="0.05" length="0.04"/>
+            </geometry>
+        </collision>
+        <xacro:inertial_cylinder mass="0.1" length="0.04" radius="0.05">
+            <origin xyz="0.0 0.0 0.0" rpy="0.0 0.0 0.0"/>
+        </xacro:inertial_cylinder>
     </link>
+    <gazebo reference="left_wheel">
+        <material>Gazebo/Black</material>
+    </gazebo>
     <joint name="right_wheel_joint" type="continuous">
-        <parent link="base_link"/>
+        <parent link="chassis"/>
         <child link="right_wheel"/>
-        <origin xyz="0.0 -0.175 0.0" rpy="${pi/2} 0.0 0.0"/>
+        <origin xyz="0.03 -0.175 0.0" rpy="${pi/2} 0.0 0.0"/>
         <axis xyz="0.0 0.0 -1"/>
     </joint>
@@ -68,4 +95,67 @@
             <material name="blue" />
         </visual>
+        <collision>
+            <geometry>
+                <cylinder radius="0.05" length="0.04"/>
+            </geometry>
+        </collision>
+        <xacro:inertial_cylinder mass="0.1" length="0.04" radius="0.05">
+            <origin xyz="0.0 0.0 0.0" rpy="0.0 0.0 0.0"/>
+        </xacro:inertial_cylinder>
     </link>
+    <gazebo reference="right_wheel">
+        <material>Gazebo/Black</material>
+    </gazebo>
+    <!-- Front left wheel joint -->
+  <joint name="front_left_wheel_joint" type="continuous">
+    <parent link="base_link" />
+    <child link="front_left_wheel" />
+    <origin xyz="0.15 0.17 0.0" rpy="-${pi/2} 0 0" />
+    <axis xyz="0 0 1" />
+  </joint>
+  <link name="front_left_wheel">
+    <visual>
+      <geometry>
+        <cylinder radius="0.05" length="0.04" />
+      </geometry>
+      <material name="blue" />
+    </visual>
+    <collision>
+      <geometry>
+        <cylinder radius="0.05" length="0.04" />
+      </geometry>
+    </collision>
+    <xacro:inertial_cylinder mass="0.1" length="0.04" radius="0.05">
+      <origin xyz="0 0 0" rpy="0 0 0" />
+    </xacro:inertial_cylinder>
+  </link>
+  <gazebo reference="front_left_wheel">
+    <material>Gazebo/Black</material>
+  </gazebo>
+  <!-- Front right wheel joint -->
+  <joint name="front_right_wheel_joint" type="continuous">
+    <parent link="base_link" />
+    <child link="front_right_wheel" />
+    <origin xyz="0.15 -0.17 0.0" rpy="${pi/2} 0 0" />
+    <axis xyz="0 0 1" />
+  </joint>
+  <link name="front_right_wheel">
+    <visual>
+      <geometry>
+        <cylinder radius="0.05" length="0.04" />
+      </geometry>
+      <material name="blue" />
+    </visual>
+    <collision>
+      <geometry>
+        <cylinder radius="0.05" length="0.04" />
+      </geometry>
+    </collision>
+    <xacro:inertial_cylinder mass="0.1" length="0.04" radius="0.05">
+      <origin xyz="0 0 0" rpy="0 0 0" />
+    </xacro:inertial_cylinder>
+  </link>
+  <gazebo reference="front_right_wheel">
+    <material>Gazebo/Black</material>
+  </gazebo>
 </robot>

Commit message: simulation

File: description/robot.urdf.xacro (robot description, xacro)
@@ -1,4 +1,6 @@
 <?xml version="1.0"?>
 <robot xmlns:xacro="http://www.ros.org/wiki/xacro"  name="robot">
-<xacro:include filename="SolidworksDesign.xacro" />
+<xacro:include filename="robot2.xacro" />
+<xacro:include filename="gazebo_control.xacro" />
+<xacro:include filename="lidar.xacro" />
 </robot>

File: description/robot_core.xacro (robot description, xacro)
@@ -31,14 +31,14 @@
     <link name="base_link">
     </link>
-    <joint name="chassis_join" type="fixed">
+    <joint name="chassis_joint" type="fixed">
         <parent link="base_link"/>
         <child link="chassis"/>
-        <origin xyz="-0.1 0.0 0.0" rpy="0.0 0.0 0.0"/>
+        <origin xyz="-0.5 0.0 0.0" rpy="0.0 0.0 0.0"/>
     </joint>
     <link name="chassis">
         <visual>
-            <origin xyz="0.15 0.0 0.075" rpy="0.0 0.0 0.0"/>
-            <geometry>
-              <mesh filename="package://firefighting_robot/meshes/base_link.STL" scale="1.0"/>
+            <origin xyz="0.5 0.0 0.17" rpy="0.0 0.0 0.0"/>
+            <geometry>
+                <box size="1 0.5 0.34"/>
             </geometry>
             <material name="pink"/>
@@ -57,8 +57,60 @@
         <material>Gazebo/Red</material>
     </gazebo>
+    <joint name="2nd floor" type="fixed">
+      <parent link="chassis"/>
+      <child link="2nd floor"/>
+      <origin xyz="0 0 0.34" rpy="0 0.0 0.0"/>
+  </joint>
+  <link name="2nd floor">
+      <visual>
+          <origin xyz="0.25 0.0 0.17" rpy="0.0 0.0 0.0"/>
+          <geometry>
+              <box size="0.5 0.5 0.34"/>
+          </geometry>
+          <material name="gray"/>
+      </visual>
+      <collision>
+          <origin xyz="0 0.0 0.0" rpy="0.0 0.0 0.0"/>
+          <geometry>
+              <box size="1 0.5 0.34"/>
+          </geometry>
+      </collision>
+      <xacro:inertial_box mass="0.5" x="0.3" y="0.3" z="0.15">
+          <origin xyz="0.15 0.0 0.075" rpy="0.0 0.0 0.0"/>
+      </xacro:inertial_box>
+  </link>
+  <gazebo reference="2nd floor">
+      <material>Gazebo/Black</material>
+  </gazebo>
+ <joint name="mechanism" type="fixed">
+        <parent link="2nd floor"/>
+        <child link="mechanism"/>
+        <origin xyz="0.5 0 0.0" rpy="0 0.0 0.0"/>
+    </joint>
+    <link name="mechanism">
+        <visual>
+            <origin xyz="0.25 0.0 0.17" rpy="0.0 0.0 0.0"/>
+            <geometry>
+                <box size="0.5 0.10 0.34"/>
+            </geometry>
+            <material name="gray2"/>
+        </visual>
+        <collision>
+            <origin xyz="0 0.0 0.0" rpy="0.0 0.0 0.0"/>
+            <geometry>
+                <box size="1 0.5 0.34"/>
+            </geometry>
+        </collision>
+        <xacro:inertial_box mass="0.5" x="0.3" y="0.3" z="0.15">
+            <origin xyz="0.15 0.0 0.075" rpy="0.0 0.0 0.0"/>
+        </xacro:inertial_box>
+    </link>
+    <gazebo reference="mechanism">
+        <material>Gazebo/GreyLight</material>
+    </gazebo>
     <joint name="left_wheel_joint" type="continuous">
         <parent link="chassis"/>
         <child link="left_wheel"/>
-        <origin xyz="0.03 0.175 0.0" rpy="-${pi/2} 0.0 0.0"/>
+        <origin xyz="0.125 0.29125 0.0" rpy="-${pi/2} 0.0 0.0"/>
         <axis xyz="0.0 0.0 1"/>
     </joint>
@@ -66,5 +118,5 @@
         <visual>
             <geometry>
-                <cylinder radius="0.05" length="0.04"/>
+                <cylinder radius="0.125" length="0.0825"/>
             </geometry>
             <material name="blue" />
@@ -85,5 +137,5 @@
         <parent link="chassis"/>
         <child link="right_wheel"/>
-        <origin xyz="0.03 -0.175 0.0" rpy="${pi/2} 0.0 0.0"/>
+        <origin xyz="0.125 -0.29125 0.0" rpy="${pi/2} 0.0 0.0"/>
         <axis xyz="0.0 0.0 -1"/>
     </joint>
@@ -91,5 +143,5 @@
         <visual>
             <geometry>
-                <cylinder radius="0.05" length="0.04"/>
+                <cylinder radius="0.125" length="0.0825"/>
             </geometry>
             <material name="blue" />
@@ -108,8 +160,8 @@
     </gazebo>
     <!-- Front left wheel joint -->
-  <joint name="front_left_wheel_joint" type="continuous">
+    <joint name="front_left_wheel_joint" type="continuous">
     <parent link="base_link" />
     <child link="front_left_wheel" />
-    <origin xyz="0.15 0.17 0.0" rpy="-${pi/2} 0 0" />
+    <origin xyz="0.375 0.29125 0.0" rpy="${pi/2} 0 0" />
     <axis xyz="0 0 1" />
   </joint>
@@ -117,5 +169,5 @@
     <visual>
       <geometry>
-        <cylinder radius="0.05" length="0.04" />
+        <cylinder radius="0.125" length="0.0825" />
       </geometry>
       <material name="blue" />
@@ -137,5 +189,5 @@
     <parent link="base_link" />
     <child link="front_right_wheel" />
-    <origin xyz="0.15 -0.17 0.0" rpy="${pi/2} 0 0" />
+    <origin xyz="0.375 -0.29125 0.0" rpy="${pi/2} 0 0" />
     <axis xyz="0 0 1" />
   </joint>
@@ -143,5 +195,5 @@
     <visual>
       <geometry>
-        <cylinder radius="0.05" length="0.04" />
+        <cylinder radius="0.125" length="0.0825" />
       </geometry>
       <material name="blue" />
