Commit message: ros2_control

File: description/lidar.xacro (robot description, xacro)
@@ -46,5 +46,5 @@
     </link>
     <gazebo reference="laser_frame">
-        <material>Gazebo/Orange</material>
+        <material>Gazebo/Black</material>
         <sensor name="laser" type="ray">
             <pose> 0 0 0 0 0 0 </pose>

File: description/robot2.xacro (robot description, xacro)
@@ -29,5 +29,5 @@
     </link>
     <gazebo reference="chassis">
-        <material>Gazebo/Wight</material>
+        <material>Gazebo/Red</material>
     </gazebo>
     <joint name="2nd floor" type="fixed">
@@ -55,5 +55,5 @@
     </link>
     <gazebo reference="2nd floor">
-        <material>Gazebo/White</material>
+        <material>Gazebo/Red</material>
     </gazebo>
     <joint name="mechanism" type="fixed">
@@ -81,5 +81,5 @@
     </link>
     <gazebo reference="mechanism">
-        <material>Gazebo/GreyLight</material>
+        <material>Gazebo/Black</material>
     </gazebo>
     <!-- Front left wheel joint -->

File: description/ros2_control.xacro (robot description, xacro)
@@ -2,5 +2,5 @@
 <robot xmlns:xacro="http://www.ros.org/wiki/xacro">
                             <!-- Real Robot -->
-    <ros2_control name="RealRobot" type="system">
+    <!-- <ros2_control name="RealRobot" type="system">
         <hardware>
             <plugin>diffdrive_arduino/DiffDriveArduino</plugin>
@@ -29,7 +29,7 @@
             <state_interface name="position"/>
         </joint>
-    </ros2_control>
+    </ros2_control> -->
                     <!-- Gazebo -->
-    <!-- <ros2_control name="GazeboSystem" type="system">
+    <ros2_control name="GazeboSystem" type="system">
         <hardware>
             <plugin>gazebo_ros2_control/GazeboSystem</plugin>
@@ -51,5 +51,5 @@
             <state_interface name="position"/>
         </joint>
-    </ros2_control> -->
+    </ros2_control>
     <gazebo>
         <plugin name="gazebo_ros2_control" filename="libgazebo_ros2_control.so">
